Commit message: [modify] gripper is not correctly set up

File: denso_robot_descriptions/vs087_description/vs087_and_robotiq/vs087_and_robotiq.urdf.xacro (robot description, xacro)
@@ -241,6 +241,6 @@
   </gazebo>
   <joint name="gripper_joint" type="fixed">
-    <origin xyz="0 0 0.038" rpy="${pi/2} 0 ${pi}"/>
-    <!-- <origin xyz="0 0 0.038" rpy="${pi/2} 0 0"/> -->
+    <!-- <origin xyz="0 0 0.038" rpy="${pi/2} 0 ${pi}"/> -->
+    <origin xyz="0 0 0.038" rpy="${pi/2} 0 0"/>
   <parent link="J6"/>
   <child link="palm"/>
@@ -252,30 +252,30 @@
   <!-- </plugin> -->
   <!-- </gazebo> -->
-  <gazebo>
-    <plugin name="gazebo_grasp_fix" filename="libgazebo_grasp_fix.so">
-      <arm>
-        <arm_name>vs087_</arm_name>
-        <palm_link>J6</palm_link>
-        <gripper_link>palm</gripper_link>
-        <gripper_link>finger_1_link_0</gripper_link>
-        <gripper_link>finger_1_link_1</gripper_link>
-        <gripper_link>finger_1_link_2</gripper_link>
-        <gripper_link>finger_1_link_3</gripper_link>
-        <gripper_link>finger_2_link_0</gripper_link>
-        <gripper_link>finger_2_link_1</gripper_link>
-        <gripper_link>finger_2_link_2</gripper_link>
-        <gripper_link>finger_middle_link_0</gripper_link>
-        <gripper_link>finger_middle_link_1</gripper_link>
-        <gripper_link>finger_middle_link_2</gripper_link>
-        <gripper_link>finger_middle_link_3</gripper_link>
-      </arm>
-      <forces_angle_tolerance>100</forces_angle_tolerance>
-      <update_rate>4</update_rate>
-      <grip_count_threshold>4</grip_count_threshold>
-      <max_grip_count>8</max_grip_count>
-      <release_tolerance>0.003</release_tolerance>
-      <disable_collisions_on_attach>false</disable_collisions_on_attach>
-      <contact_topic>__default_topic__</contact_topic>
-    </plugin>
-  </gazebo>
+  <!-- <gazebo> -->
+  <!--   <plugin name="gazebo_grasp_fix" filename="libgazebo_grasp_fix.so"> -->
+  <!--     <arm> -->
+  <!--       <arm_name>vs087_</arm_name> -->
+  <!--       <palm_link>J6</palm_link> -->
+  <!--       <gripper_link>palm</gripper_link> -->
+  <!--       <gripper_link>finger_1_link_0</gripper_link> -->
+  <!--       <gripper_link>finger_1_link_1</gripper_link> -->
+  <!--       <gripper_link>finger_1_link_2</gripper_link> -->
+  <!--       <gripper_link>finger_1_link_3</gripper_link> -->
+  <!--       <gripper_link>finger_2_link_0</gripper_link> -->
+  <!--       <gripper_link>finger_2_link_1</gripper_link> -->
+  <!--       <gripper_link>finger_2_link_2</gripper_link> -->
+  <!--       <gripper_link>finger_middle_link_0</gripper_link> -->
+  <!--       <gripper_link>finger_middle_link_1</gripper_link> -->
+  <!--       <gripper_link>finger_middle_link_2</gripper_link> -->
+  <!--       <gripper_link>finger_middle_link_3</gripper_link> -->
+  <!--     </arm> -->
+  <!--     <forces_angle_tolerance>100</forces_angle_tolerance> -->
+  <!--     <update_rate>4</update_rate> -->
+  <!--     <grip_count_threshold>4</grip_count_threshold> -->
+  <!--     <max_grip_count>8</max_grip_count> -->
+  <!--     <release_tolerance>0.003</release_tolerance> -->
+  <!--     <disable_collisions_on_attach>false</disable_collisions_on_attach> -->
+  <!--     <contact_topic>__default_topic__</contact_topic> -->
+  <!--   </plugin> -->
+  <!-- </gazebo> -->
 </robot>
